File: vortex-numpad.kicad_pcb (KiCad board)
At the start: 2 copper layers, 0 parts

Commit message: Initial PCB layout
Parts:
- added ASTERISK1: MX-NoLED, MX_Alps_Hybrid:MX-1U-NoLED, F.Cu at (115.9, 94.5)
- added C1: 1uF, Diode_SMD:D_SOD-123, B.Cu at (123.8, 85.7)
- added C2: 1uF, Diode_SMD:D_SOD-123, B.Cu at (123.8, 82.5)
- added C3: 1uF, Diode_SMD:D_SOD-123, B.Cu at (119.1, 77.0)
- added C4: 0.1uF, Diode_SMD:D_SOD-123, B.Cu at (87.3, 85.7)
- added C5: 0.1uF, Diode_SMD:D_SOD-123, B.Cu at (92.1, 84.1)
- added C6: 0.1uF, Diode_SMD:D_SOD-123, B.Cu at (88.9, 77.0)
- added C7: 10uF, Diode_SMD:D_SOD-123, B.Cu at (87.3, 82.5)
- added D1: SOD-123, Diode_SMD:D_SOD-123, B.Cu at (81.0, 77.0)
- added D10: SOD-123, Diode_SMD:D_SOD-123, B.Cu at (104.8, 113.5)
- added D11: SOD-123, Diode_SMD:D_SOD-123, B.Cu at (123.8, 117.5)
- added D12: SOD-123, Diode_SMD:D_SOD-123, B.Cu at (85.7, 132.6)
- added D13: SOD-123, Diode_SMD:D_SOD-123, B.Cu at (104.8, 132.6)
- added D14: SOD-123, Diode_SMD:D_SOD-123, B.Cu at (123.8, 128.6)
- added D15: SOD-123, Diode_SMD:D_SOD-123, B.Cu at (127.8, 128.6)
- added D16: SOD-123, Diode_SMD:D_SOD-123, B.Cu at (85.7, 151.6)
- added D17: SOD-123, Diode_SMD:D_SOD-123, B.Cu at (104.8, 151.6)
- added D18: SOD-123, Diode_SMD:D_SOD-123, B.Cu at (123.8, 155.6)
- added D19: SOD-123, Diode_SMD:D_SOD-123, B.Cu at (85.7, 170.7)
- added D2: SOD-123, Diode_SMD:D_SOD-123, B.Cu at (93.7, 77.0)
- added D20: SOD-123, Diode_SMD:D_SOD-123, B.Cu at (104.8, 170.7)
- added D21: SOD-123, Diode_SMD:D_SOD-123, B.Cu at (123.8, 166.7)
- added D22: SOD-123, Diode_SMD:D_SOD-123, B.Cu at (127.8, 166.7)
- added D3: SOD-123, Diode_SMD:D_SOD-123, B.Cu at (123.8, 72.2)
- added D4: SOD-123, Diode_SMD:D_SOD-123, B.Cu at (142.9, 72.2)
- added D5: SOD-123, Diode_SMD:D_SOD-123, B.Cu at (85.7, 94.5)
- added D6: SOD-123, Diode_SMD:D_SOD-123, B.Cu at (104.8, 94.5)
- added D7: SOD-123, Diode_SMD:D_SOD-123, B.Cu at (123.8, 94.5)
- added D8: SOD-123, Diode_SMD:D_SOD-123, B.Cu at (142.9, 94.5)
- added D9: SOD-123, Diode_SMD:D_SOD-123, B.Cu at (85.7, 113.5)
- added F1: 500mA, Fuse:Fuse_1206_3216Metric, B.Cu at (85.7, 77.0)
- added FN1: MX-NoLED, MX_Alps_Hybrid:MX-1U-NoLED, F.Cu at (77.8, 72.2)
- added FN2: MX-NoLED, MX_Alps_Hybrid:MX-1U-NoLED, F.Cu at (96.8, 72.2)
- added FN3: MX-NoLED, MX_Alps_Hybrid:MX-1U-NoLED, F.Cu at (115.9, 72.2)
- added FN4: MX-NoLED, MX_Alps_Hybrid:MX-1U-NoLED, F.Cu at (134.9, 72.2)
- added FWDSLASH1: MX-NoLED, MX_Alps_Hybrid:MX-1U-NoLED, F.Cu at (96.8, 94.5)
- added J1: USB_B_Micro, Connector_USB:USB_Micro-B_Molex-105017-0001, B.Cu at (87.3, 65.4)
- added MINUS1: MX-NoLED, MX_Alps_Hybrid:MX-1U-NoLED, F.Cu at (134.9, 94.5)
- added NUM0: MX-NoLED, MX_Alps_Hybrid:MX-1U-NoLED, F.Cu at (77.8, 170.7)
- added NUM1: MX-NoLED, MX_Alps_Hybrid:MX-1U-NoLED, F.Cu at (77.8, 151.6)
- added NUM2: MX-NoLED, MX_Alps_Hybrid:MX-1U-NoLED, F.Cu at (96.8, 151.6)
- added NUM3: MX-NoLED, MX_Alps_Hybrid:MX-1U-NoLED, F.Cu at (115.9, 151.6)
- added NUM4: MX-NoLED, MX_Alps_Hybrid:MX-1U-NoLED, F.Cu at (77.8, 132.6)
- added NUM5: MX-NoLED, MX_Alps_Hybrid:MX-1U-NoLED, F.Cu at (96.8, 132.6)
- added NUM6: MX-NoLED, MX_Alps_Hybrid:MX-1U-NoLED, F.Cu at (115.9, 132.6)
- added NUM7: MX-NoLED, MX_Alps_Hybrid:MX-1U-NoLED, F.Cu at (77.8, 113.5)
- added NUM8: MX-NoLED, MX_Alps_Hybrid:MX-1U-NoLED, F.Cu at (96.8, 113.5)
- added NUM9: MX-NoLED, MX_Alps_Hybrid:MX-1U-NoLED, F.Cu at (115.9, 113.5)
- added NUMDBL0: MX-NoLED, MX_Alps_Hybrid:MX-1U-NoLED, F.Cu at (96.8, 170.7)
- added NUMDOT1: MX-NoLED, MX_Alps_Hybrid:MX-1U-NoLED, F.Cu at (115.9, 170.7)
- added NUMLOCK1: MX-NoLED, MX_Alps_Hybrid:MX-1U-NoLED, F.Cu at (77.8, 94.5)
- added PLUS1: MX-NoLED, MX_Alps_Hybrid:MX-2U-ReversedStabilizers-NoLED, F.Cu at (134.9, 123.0)
- added R1: 10k, Resistor_SMD:R_0805_2012Metric, B.Cu at (74.5, 85.6)
- added R2: 22, Resistor_SMD:R_0805_2012Metric, B.Cu at (74.5, 82.6)
- added R3: 22, Resistor_SMD:R_0805_2012Metric, B.Cu at (74.5, 79.7)
- added R4: 10k, Resistor_SMD:R_0805_2012Metric, B.Cu at (74.5, 76.7)
- added RETURN1: MX-NoLED, MX_Alps_Hybrid:MX-2U-ReversedStabilizers-NoLED, F.Cu at (134.9, 161.1)
- added SW1: SW_Push, random-keyboard-parts:SKQG-1155865, B.Cu at (134.9, 81.0)
- added U1: ATmega32U4-AU, Package_QFP:TQFP-44_10x10mm_P0.8mm, B.Cu at (106.4, 81.0)
- added Y1: 16MHz, Crystal:Crystal_SMD_3225-4Pin_3.2x2.5mm, B.Cu at (117.5, 84.3)
Other:
- board outline added: 76.2 x 117.5 mm
